Commit message: Add files to detect and segment images. Update the static camera's XACRO file to set its location/pose.

File: urdf/static_zed2_camera.xacro (robot description, xacro)
@@ -1,9 +1,7 @@
 <?xml version="1.0"?>
 <robot xmlns:xacro="http://www.ros.org/wiki/xacro" name="static_zed2_camera">
-    <!-- <joint name="zed2_holder_joint" type="fixed">
-        <parent link="panda_hand"/>
-        <child link="zed2_holder"/>
-        <origin xyz="0 0 0" rpy="${pi} 0 0"/>
-    </joint> -->
+    <gazebo>
+        <static>false</static>
+    </gazebo>
     <!-- 1. DUMMY ROOT LINK (The "World" anchor for this model) -->
     <link name="world_interface_link"/>
@@ -30,4 +28,8 @@
         </visual>
     </link>
+    <!-- Disable gravity for camera holder -->
+    <gazebo reference="static_zed2_holder">
+        <gravity>false</gravity>
+    </gazebo>
     <joint name="camera_joint" type="fixed">
         <parent link="static_zed2_holder"/>
@@ -56,4 +58,8 @@
         </collision>
     </link>
+    <!-- Disable gravity for main camera link -->
+    <gazebo reference="static_zed2_camera_link">
+        <gravity>false</gravity>
+    </gazebo>
     <!-- Left Camera -->
     <joint name="left_camera_joint" type="fixed">
@@ -85,4 +91,5 @@
     <gazebo reference="static_zed2_left_camera_link">
     <!-- Raw images (with lens distortion) -->
+        <gravity>false</gravity>
         <material>Gazebo/Red</material>
         <sensor name="static_zed2_left_raw_camera" type="camera">
@@ -176,4 +183,5 @@
     <gazebo reference="static_zed2_right_camera_link">
     <!-- Raw images (with lens distortion) -->
+        <gravity>false</gravity>
         <sensor name="static_zed2_right_raw_camera" type="camera">
             <pose> 0 0 0 0 0 0 </pose>
@@ -273,6 +281,8 @@
       </sensor>
     </gazebo>
-     <gazebo>
-        <static>true</static>
-    </gazebo>
 </robot>
+    <!-- <joint name="zed2_holder_joint" type="fixed">
+        <parent link="panda_hand"/>
+        <child link="zed2_holder"/>
+        <origin xyz="0 0 0" rpy="${pi} 0 0"/>
+    </joint> -->
